File: KiCad/LastAcolyte.kicad_sch (KiCad schematic)
At the start: 86 parts, among them J1 USB_B, J2 Mini-DIN-6, J3 AudioJack3, J4 DB15_Female_HighDensity, J5 Conn-01x06, J6 Conn_01x02, J7 Conn_02x20_Odd_Even, Q1 PN2222A, SW1 SW_SPDT, SW2 SW_Push, U1 W65C02SxP, U10 74HC273, U11 74HC166, U12 74HC166, U13 74HC10, U14 74HC00, U15 74HC02, U16 MCP130-xxxDxTO, U17 25LCxxx, U18 W65C22SxP, U19 74HC688, U2 AS6C4008-55PCN, U20 74HC08, U3 SST39SF040, U4 74HC161, U5 74HC590, U6 74HC590, U7 74HC590, U8 74HC245, U9 74HC377, X1 CXO_DIP8/14

Commit message: Add files via upload
Parts:
- removed C23, C24: C, Capacitor_THT:C_Disc_D5.0mm_W2.5mm_P5.00mm, symbol Device:C
- removed JP3, JP4: SolderJumper_2_Open, Library:SolderJumper_Testing-2_P1.3mm_Open_Pad1.0x1.5mm, symbol Jumper:SolderJumper_2_Open
- removed R19: R_US, Resistor_THT:R_Axial_DIN0207_L6.3mm_D2.5mm_P7.62mm_Horizontal, symbol Device:R_US
- removed U18: W65C22SxP, Package_DIP:DIP-40_W15.24mm_Socket, symbol 65xx:W65C22SxP
- removed U19: 74HC688, Package_DIP:DIP-20_W7.62mm_Socket, symbol 74xx:74HC688
- renumbered R18 to R15, R15 to R16, R16 to R18, U20 to U14, U14 to U15, U15 to U16, U16 to U17, U17 to U18
Connections:
- net +5V: now also U15.1; no longer U14.4, U14.5, U15.4
- net A0: now also J7.4 (Pin_4)
- net A1: now also J7.6 (Pin_6)
- net A10: now also J7.28 (Pin_28)
- net A11: now also J7.30 (Pin_30)
- net A12: now also J7.32 (Pin_32)
- net A13: now also J7.34 (Pin_34)
- net A14: now also J7.36 (Pin_36), U14.13
- net A15: now also J7.38 (Pin_38), U13.10, U14.12; no longer U15.1
- net A2: now also J7.8 (Pin_8)
- net A3: now also J7.10 (Pin_10)
- net A4: now also J7.12 (Pin_12)
- net A5: now also J7.14 (Pin_14)
- net A6: now also J7.16 (Pin_16)
- net A7: now also J7.18 (Pin_18)
- net A8: now also J7.24 (Pin_24)
- net A9: now also J7.26 (Pin_26)
- net CA1: no longer J7.31 (Pin_31)
- net CA2: no longer J7.33 (Pin_33)
- net CB1: no longer J7.35 (Pin_35)
- net CB2: no longer J7.37 (Pin_37)
- net D0: now also J7.23 (Pin_23); no longer J7.3 (Pin_3)
- net D1: now also J7.25 (Pin_25); no longer J7.5 (Pin_5)
- net D2: now also J7.27 (Pin_27); no longer J7.7 (Pin_7)
- net D3: now also J7.29 (Pin_29); no longer J7.9 (Pin_9)
- net D4: now also J7.31 (Pin_31); no longer J7.11 (Pin_11)
- net D5: now also J7.33 (Pin_33); no longer J7.13 (Pin_13)
- net D6: now also J7.35 (Pin_35); no longer J7.15 (Pin_15)
- net D7: now also J7.37 (Pin_37); no longer J7.17 (Pin_17)
- net HIGH: now also U14.11, U15.4; no longer U13.4, U15.6
- net LAST: now also J7.9 (Pin_9), U13.3
- net PA0: no longer J7.4 (Pin_4)
- net PA1: no longer J7.6 (Pin_6)
- net PA2: no longer J7.8 (Pin_8)
- net PA3: no longer J7.10 (Pin_10)
- net PA4: no longer J7.12 (Pin_12)
- net PA5: no longer J7.14 (Pin_14)
- net PA6: no longer J7.16 (Pin_16)
- net PA7: no longer J7.18 (Pin_18)
- net PB0: no longer J7.24 (Pin_24)
- net PB1: no longer J7.26 (Pin_26)
- net PB2: no longer J7.28 (Pin_28)
- net PB3: no longer J7.30 (Pin_30)
- net PB4: no longer J7.32 (Pin_32)
- net PB5: no longer J7.34 (Pin_34)
- net PB6: no longer J7.36 (Pin_36)
- net PB7: no longer J7.38 (Pin_38)
- net PHI2: now also U15.9; no longer U13.10, U13.3, U15.10
- net QUARTER: no longer U13.11
- net RDY: now also J7.5 (Pin_5)
- net SIXTEENTH: now also U15.13; no longer U15.12
- net SYNC: now also J7.3 (Pin_3); no longer J7.27 (Pin_27)
- net ~{IO}: now also J7.13 (Pin_13), U13.8, U14.4; no longer J7.29 (Pin_29), U14.12
- net ~{OE}: now also U13.4, U15.5; no longer U13.5, U13.9
- net ~{OUTPUT}: now also U15.6; no longer U13.6
- net ~{PHI2}: now also U16.12; no longer J7.25 (Pin_25), U16.11
- net ~{RES}: now also J7.7 (Pin_7)
- net ~{ROM}: now also U14.5, U15.10; no longer U15.9
- net ~{RW}: now also J7.15 (Pin_15); no longer J7.23 (Pin_23)
- net ~{SPI-MISO}: now also U15.12; no longer U15.13
- net ~{WE}: now also U13.6; no longer U13.8
- net RAMADDR: now reaches U14.6
- net RAMADDR: now also U13.5, U16.11
- net BANK-A renamed BANK-ROM
- net BANK-B renamed BANK-RAM
- net RBK renamed RAMEXP
- removed net RCE: U14.11, U16.12
- net VIA-ENABLE renamed IO-ENABLE
- net IO-ENABLE: now also J7.11 (Pin_11), U13.11
- net VIA-INT renamed IO-INT
- net IO-INT: now also J7.17 (Pin_17)
- removed net ~{HIGH}: U14.13, U15.3, U15.5
- new net ~{A14}: U13.9, U15.3
- no-connect marks 27 -> 26
Other:
- note added: "CS1"
- note added: "D0"
- note added: "D1"
- note added: "D2"
- note added: "D3"
- note added: "D4"
- note added: "D5"
- note added: "D6"
- note added: "D7"
- note added: "Expected VIA expansion. Must be enabled through software."
- note added: "Memory Map: $0000-$07FF = RAM $0800-$7FFF = Video RAM $8000-$BFFF = RAM or I/O $C000-$FFFF = ROM (banked)"
- note added: "PHI2"
- note added: "R/~{W}"
- note added: "RS0"
- note added: "RS1"
- note added: "RS2"
- note added: "RS3"
- note added: "W65C22SxP"
- note added: "~{CS2}"
- note added: "~{IRQ}"
- note added: "~{RES}"
- note removed: "KEY-INT"
- note removed: "Memory Map: $0000-$07FF = RAM $0800-$7FFF = Video RAM $8000-$BEFF = RAM (banked) $BF00-$BFFF = I/O Expansion $C000-$FFFF = ROM (banked)"
- note removed: "RAM-ADDR"
- note removed: "VIA Expansion (optional)"
- note removed: "VIA must be enabled through software."
- moved on the sheet: C10, C11, C12, C13, C14, C15, C16, C17, C18, C19, C2, C20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

Commit message: Add files via upload
Connections:
- net IO-ENABLE: no longer J7.11 (Pin_11)
- net PHI2: now also J7.11 (Pin_11)
Changed lines of the file:
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@@
     )
   )
-  (global_label "IO-ENABLE" (shape input) (at 137.16 364.49 180) (fields_autoplaced)
-    (effects (font (size 1.27 1.27)) (justify right))
-    (property "Intersheet References" "${INTERSHEET_REFS}" (id 0) (at 126.9455 364.4106 0)
+  (global_label "PHI2" (shape input) (at 137.16 364.49 180) (fields_autoplaced)
+    (effects (font (size 1.27 1.27)) (justify right))
+    (property "Intersheet References" "${INTERSHEET_REFS}" (id 0) (at 130.3321 364.4106 0)
       (effects (font (size 1.27 1.27)) (justify right) hide)
     )
@@
     )
   )
-  (global_label "IO-ENABLE" (shape input) (at 228.6 344.17 180) (fields_autoplaced)
-    (effects (font (size 1.27 1.27)) (justify right))
-    (property "Intersheet References" "${INTERSHEET_REFS}" (id 0) (at 218.3855 344.0906 0)
+  (global_label "PHI2" (shape input) (at 228.6 344.17 180) (fields_autoplaced)
+    (effects (font (size 1.27 1.27)) (justify right))
+    (property "Intersheet References" "${INTERSHEET_REFS}" (id 0) (at 221.7721 344.0906 0)
       (effects (font (size 1.27 1.27)) (justify right) hide)
     )
@@
   )
   (symbol (lib_id "power:+5V") (at 212.09 31.75 0) (unit 1)
-    (in_bom yes) (on_board yes) (fields_autoplaced)
+    (in_bom yes) (on_board yes)
     (property "Reference" "#PWR0192" (id 0) (at 212.09 35.56 0)
       (effects (font (size 1.27 1.27)) hide)
@@
   )
   (symbol (lib_id "Power_Supervisor:MCP130-xxxDxTO") (at 118.11 177.8 0) (unit 1)
-    (in_bom yes) (on_board yes) (fields_autoplaced)
+    (in_bom yes) (on_board yes)
     (property "Reference" "U17" (id 0) (at 111.76 176.5299 0)
       (effects (font (size 1.27 1.27)) (justify right))

Commit message: Add files via upload
Parts:
- added Q2, Q3: PN2222A, Package_TO_SOT_THT:TO-92_HandSolder, symbol Transistor_BJT:PN2222A
- added R19: R_US, Resistor_THT:R_Axial_DIN0207_L6.3mm_D2.5mm_P7.62mm_Horizontal, symbol Device:R_US
Connections:
- net +5V: now also R19.1
- net GND: now also Q2.1 (E)
- net SPI-MISO: now also Q3.1 (E); no longer J5.3 (Pin_3)
- net SPI-SDCARD: now also Q2.2 (B)
- new net SPI-SDCARD-MISO: J5.3 (Pin_3), Q3.3 (C)
- new net ~{SPI-SDCARD}: Q2.3 (C), Q3.2 (B), R19.2
Other:
- note added: "$0000"
- note added: "$0800"
- note added: "$8000"
- note added: "$8380"
- note added: "0"
- note added: "1"
- note added: "Horizontal Back Porch"
- note added: "Horizontal Front Porch"
- note added: "Horizontal Sync"
- note added: "Odd Parity=?"
- note added: "Reading from RAM"
- note added: "Reading from ROM"
- note added: "Start Bit=0"
- note added: "Stop Bit=1"
- note added: "Vertical Back Porch"
- note added: "Vertical Front Porch"
- note added: "Vertical Sync"
- note added: "Video"
- note added: "Visible Area"
- note added: "Writing to RAM"
- note added: "Writing to ROM (causes Output)"
- moved on the sheet: Q1, R17, U15D

Commit message: Add files via upload
Parts:
- R6: Field4 10k -> 3.3k
Connections:
- net +5V: now also R15.2, R8.2; no longer R15.1, R8.1
- net IO-INT: now also R15.1; no longer R15.2
- net SPI-MISO: now also R8.1; no longer R8.2
Other:
- note added: "Read Byte"
- note added: "Read Command"
- note added: "Upper/Lower Addresses"
- note added: "Write Byte"
- note added: "Write Command"
- moved on the sheet: C2, D2, D3, J2, J3, J5, Q1, Q2, Q3, R15, R16, R17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

Commit message: Add files via upload
Connections:
- net A0: now also J7.23 (Pin_23); no longer J7.4 (Pin_4)
- net A1: now also J7.25 (Pin_25); no longer J7.6 (Pin_6)
- net A2: now also J7.27 (Pin_27); no longer J7.8 (Pin_8)
- net A3: now also J7.29 (Pin_29); no longer J7.10 (Pin_10)
- net A4: now also J7.31 (Pin_31); no longer J7.12 (Pin_12)
- net A5: now also J7.33 (Pin_33); no longer J7.14 (Pin_14)
- net A6: now also J7.35 (Pin_35); no longer J7.16 (Pin_16)
- net A7: now also J7.37 (Pin_37); no longer J7.18 (Pin_18)
- net C0: now also J7.4 (Pin_4)
- net C1: now also J7.6 (Pin_6)
- net C2: now also J7.8 (Pin_8)
- net C3: now also J7.10 (Pin_10)
- net C4: now also J7.12 (Pin_12)
- net C5: now also J7.14 (Pin_14)
- net C6: now also J7.16 (Pin_16)
- net C7: now also J7.18 (Pin_18)
- net D0: no longer J7.23 (Pin_23)
- net D1: no longer J7.25 (Pin_25)
- net D2: no longer J7.27 (Pin_27)
- net D3: no longer J7.29 (Pin_29)
- net D4: no longer J7.31 (Pin_31)
- net D5: no longer J7.33 (Pin_33)
- net D6: no longer J7.35 (Pin_35)
- net D7: no longer J7.37 (Pin_37)
Other:
- note added: "Acolyte Computer Steven Chad Burrow 2023, Public Domain W65C02 running at 3.14 MHz 2KB System RAM 30KB Video RAM 16KB Banked RAM (up to 2 banks) 16KB Banked ROM (up to 2 banks)"
- note added: "General Expansion"
- note removed: "$0000"
- note removed: "$0800"
- note removed: "$8000"
- note removed: "$8380"
- note removed: "0"
- note removed: "1"
- note removed: "Acolyte Computer Professor Steven Chad Burrow 2023, Public Domain W65C02 running at 3.14 MHz 2KB System RAM 30KB Video RAM 16KB Banked RAM (up to 2 banks) 16KB Banked ROM (up to 2 banks)"
- note removed: "Expansion"
- note removed: "Horizontal Back Porch"
- note removed: "Horizontal Front Porch"
- note removed: "Horizontal Sync"
- note removed: "Odd Parity=?"
- note removed: "Read Byte"
- note removed: "Read Command"
- note removed: "Reading from RAM"
- note removed: "Reading from ROM"
- note removed: "Start Bit=0"
- note removed: "Stop Bit=1"
- note removed: "Upper/Lower Addresses"
- note removed: "Vertical Back Porch"
- note removed: "Vertical Front Porch"
- note removed: "Vertical Sync"
- note removed: "Video"
- note removed: "Visible Area"
- note removed: "Write Byte"
- note removed: "Write Command"
- note removed: "Writing to RAM"
- note removed: "Writing to ROM (causes Output)"
- note removed: "http://falstad.com/circuit/circuitjs.html?ctz=CQAgjCAMB0l3BWcMBMcUHYMGZIA4UA2ATmIxAUgpABZsKBTAWjDACgAlcFPcQqsDxDFCUMTSpIq06AjYBlcMRTgMowbzBqxEAGYBDADYBnBmJQKlK7NnVCbogSAMmzVC1w0hsabrxQIjuKSYjJyAOZ+3ggqXth4NKFskV5gylEoKInSbADuVqqiPJra7ABOIMWF3rbVVIRobBVVaLwOlfhiGJRNlXj+EjVFgwKUcHl9JUX9HbyQEy2dLSMTada1Ve3lk0O77e4S880ztm21pzpjvVWHu7eSYPP5mxsnhHMLb-4z9xNb2nRYtoLPl2q1aD5ZpU-htBoDKoMQRCgaIaDQplBemiMTQR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"
- moved on the sheet: C10, C11, C12, C13, C14, C15, C16, C17, C18, C19, C2, C20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

Commit message: Add files via upload
Parts:
- removed R15: R_US, Resistor_THT:R_Axial_DIN0207_L6.3mm_D2.5mm_P7.62mm_Horizontal, symbol Device:R_US
- added R20: R_US, Resistor_THT:R_Axial_DIN0207_L6.3mm_D2.5mm_P7.62mm_Horizontal, symbol Device:R_US
- added TP6, TP7: TestPoint, Library:CustomTestPoint, symbol Connector:TestPoint
- J7: footprint Connector_PinHeader_2.54mm:PinHeader_2x20_P2.54mm_Vertical -> Connector_PinSocket_2.54mm:PinSocket_2x20_P2.54mm_Vertical
- renumbered U9 to U10, U10 to U9
Connections:
- net +5V: now also R16.2, R20.2; no longer R16.1, U15.1
- net A0: now also J7.38 (Pin_38); no longer J7.23 (Pin_23)
- net A1: now also J7.36 (Pin_36); no longer J7.25 (Pin_25)
- net A10: now also J7.14 (Pin_14); no longer J7.28 (Pin_28)
- net A11: now also J7.12 (Pin_12); no longer J7.30 (Pin_30)
- net A12: now also U14.2; no longer J7.32 (Pin_32)
- net A13: now also U14.1; no longer J7.34 (Pin_34)
- net A14: now also U16.2; no longer J7.36 (Pin_36), U15.2
- net A15: now also U15.1; no longer D2.1 (K), J7.38 (Pin_38)
- net A2: now also J7.34 (Pin_34); no longer J7.27 (Pin_27)
- net A3: now also J7.32 (Pin_32); no longer J7.29 (Pin_29)
- net A4: now also J7.30 (Pin_30); no longer J7.31 (Pin_31)
- net A5: now also J7.28 (Pin_28); no longer J7.33 (Pin_33)
- net A6: now also J7.26 (Pin_26); no longer J7.35 (Pin_35)
- net A7: now also J7.24 (Pin_24); no longer J7.37 (Pin_37)
- net A8: now also J7.18 (Pin_18); no longer J7.24 (Pin_24)
- net A9: now also J7.16 (Pin_16); no longer J7.26 (Pin_26)
- net AUDIO-OUT: now also J7.21 (Pin_21)
- net C0: now also J7.3 (Pin_3), U8.2 (A0); no longer J7.4 (Pin_4), U8.9 (A7)
- net C1: now also J7.5 (Pin_5), U8.3 (A1); no longer J7.6 (Pin_6), U8.8 (A6)
- net C2: now also J7.7 (Pin_7), U8.4 (A2); no longer J7.8 (Pin_8), U8.7 (A5)
- net C3: now also J7.9 (Pin_9), U8.5 (A3); no longer J7.10 (Pin_10), U8.6 (A4)
- net C4: now also J7.11 (Pin_11), U8.6 (A4); no longer J7.12 (Pin_12), U8.5 (A3)
- net C5: now also J7.13 (Pin_13), U8.7 (A5); no longer J7.14 (Pin_14), U8.4 (A2)
- net C6: now also J7.15 (Pin_15), U8.8 (A6); no longer J7.16 (Pin_16), U8.3 (A1)
- net C7: now also J7.17 (Pin_17), U8.9 (A7); no longer J7.18 (Pin_18), U8.2 (A0)
- net CLK: now also J7.29 (Pin_29)
- net D0: now also U8.18 (B0); no longer U8.11 (B7)
- net D1: now also U8.17 (B1); no longer U8.12 (B6)
- net D2: now also U8.16 (B2); no longer U8.13 (B5)
- net D3: now also U8.15 (B3); no longer U8.14 (B4)
- net D4: now also U8.14 (B4); no longer U8.15 (B3)
- net D5: now also U8.13 (B5); no longer U8.16 (B2)
- net D6: now also U8.12 (B6); no longer U8.17 (B1)
- net D7: now also U8.11 (B7); no longer U8.18 (B0)
- net GND: now also TP6.1, TP7.1
- net HALF: now also J7.27 (Pin_27)
- net IO-ENABLE: now also U16.3, U9.15 (Q5); no longer U13.11, U9.16 (Q6)
- net IO-INT: now also D3.1 (K), J7.8 (Pin_8), R20.1; no longer J7.17 (Pin_17), U14.9
- net KEY-CLK: now also U14.4; no longer U14.10, U16.3
- net KEY-DATA: now also D2.1 (K); no longer U16.2
- net LAST: no longer J7.9 (Pin_9), U13.3, U14.3
- net PHI2: now also J7.23 (Pin_23); no longer J7.11 (Pin_11), U14.1
- net QUARTER: now also J7.25 (Pin_25), U13.3; no longer U14.2
- net RAMADDR: now also U14.8; no longer U14.6
- net RAMEXP: now also U15.3; no longer D2.2 (A), D3.2 (A), R16.2
- net RDY: now also J7.31 (Pin_31); no longer J7.5 (Pin_5)
- net SPI-MISO: now also J7.4 (Pin_4); no longer J7.21 (Pin_21)
- net SYNC: now also J7.37 (Pin_37); no longer J7.3 (Pin_3)
- net ~{A14}: now also U16.1; no longer U15.3
- net ~{IO}: now also J7.10 (Pin_10), U14.9; no longer J7.13 (Pin_13), U14.4
- net ~{IRQ}: now also D2.2 (A), D3.2 (A), R16.1; no longer U14.8
- net ~{NMI}: now also U14.6; no longer U16.1
- net ~{OE}: now also J7.33 (Pin_33)
- net ~{RES}: now also J7.6 (Pin_6); no longer J7.7 (Pin_7)
- net ~{ROM}: now also U14.10; no longer U14.5
- net ~{RW}: now also J7.35 (Pin_35); no longer J7.15 (Pin_15)
- net LED: now reaches D1.2 (A), R1.1
- removed net BANK-RAM: D3.1 (K), U9.15 (Q5)
- net BANK-ROM renamed MEM-BANK
- net MEM-BANK: now also U15.2
- new net MID: U13.11, U14.3
- new net NMI-ENABLE: U14.5, U9.16 (Q6)
Other:
- note added: "$0000"
- note added: "$0800"
- note added: "$8000"
- note added: "$8380"
- note added: "0"
- note added: "1"
- note added: "6522 VIA Expansion"
- note added: "Acolyte Computer Steven Chad Burrow 2023, Public Domain"
- note added: "EXPANSION"
- note added: "Horizontal Back Porch"
- note added: "Horizontal Front Porch"
- note added: "Horizontal Sync"
- note added: "Memory Map: $0000-$07FF = RAM $0800-$7FFF = Video RAM $8000-$AFFF = RAM (banked) $B000-$BFFF = I/O (or RAM) $C000-$FFFF = ROM (banked)"
- note added: "Odd Parity=?"
- note added: "Pull-up resistors"
- note added: "Read Byte"
- note added: "Read Command"
- note added: "Reading from RAM"
- note added: "Reading from ROM"
- note added: "Start Bit=0"
- note added: "Stop Bit=1"
- note added: "Upper/Lower Addresses"
- note added: "Vertical Back Porch"
- note added: "Vertical Front Porch"
- note added: "Vertical Sync"
- note added: "Video"
- note added: "Visible Area"
- note added: "W65C02 running at 3.14 MHz 2KB System RAM 30KB Video RAM 12KB Banked RAM 4KB I/O (or RAM) 16KB Banked ROM"
- note added: "Write Byte"
- note added: "Write Command"
- note added: "Writing to RAM"
- note added: "Writing to ROM (causes Output)"
- note added: "http://falstad.com/circuit/circuitjs.html?ctz=CQAgjCAMB0l3BWcMBMcUHYMGZIA4UA2ATmIxAUgpABZsKBTAWjDACgAlcFPcQqsDxDFCUMTSpIq06AjYBlcMRTgMowbzBqxEAGYBDADYBnBmJQKlK7NnVCbogSAMmzVC1w0hsabrxQIjuKSYjJyAOZ+3ggqXth4NKFskV5gylEoKInSbADuVqqiPJra7ABOIMWF3rbVVIRobBVVaLwOlfhiGJRNlXj+EjVFgwKUcHl9JUX9HbyQEy2dLSMTada1Ve3lk0O77e4S880ztm21pzpjvVWHu7eSYPP5mxsnhHMLb-4z9xNb2nRYtoLPl2q1aD5ZpU-htBoDKoMQRCgaIaDQplBemiMTQR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"
- note added: "http://falstad.com/circuit/circuitjs.html?ctz=CQAgjCAMB0l3BWcMBMcUHYMGZIA4UA2ATmIxAUgpABZsKBTAWjDACgBzEYsFEF4nx58WNGlChsA7t178UePLJFhBIbNOX8Ec4fMWSZephkJLjOvpDYAnEHhpKmC83OcGqGBLfuPtut0sJLx8HJ1NXEQjg7xlo9yUw-SUNOLN-PiSmINSQeOis6NzsB2TaPCoE9U0aQnFsuQRCSpyauv5opsqiznBTDvSwfpNsQglrGRQabsHhnoBlEBcO0qnu0qoIADMAQwAbAGcGCRRNIbGmCqo1-ivqgCU+i8VN4eIxcdoqJCpf6Finrc4IDLhVqnZCFMBkp8ukqNhcD5IfUgvEgvDERCoVV4st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"
- note removed: "Acolyte Computer Steven Chad Burrow 2023, Public Domain W65C02 running at 3.14 MHz 2KB System RAM 30KB Video RAM 16KB Banked RAM (up to 2 banks) 16KB Banked ROM (up to 2 banks)"
- note removed: "Expected VIA expansion. Must be enabled through software."
- note removed: "General Expansion"
- note removed: "Memory Map: $0000-$07FF = RAM $0800-$7FFF = Video RAM $8000-$BFFF = RAM or I/O $C000-$FFFF = ROM (banked)"
- moved on the sheet: C1, C10, C11, C12, C13, C14, C15, C16, C17, C18, C19, C2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
